File: VS1000DBreakout.sch (KiCad schematic (older format))
At the start: 1 part

Commit message: Almost copied it all
Parts:
- removed IC?: VS1000, symbol VS1000
- added C? (x6): 10uF, symbol C
- added C?: 1uF, symbol C
- added C? (x2): 4.7nF, symbol C
- added D? (x2): LED, symbol LED
- added D?: 1N4148, symbol D
- added D? (x2): MBR120, symbol ZENER
- added GPIO?: GPIO_Breakout, symbol GPIO_Breakout
- added IC?: VS1000, symbol VS1000
- added R? (x16): 100K, symbol R
- added R? (x4): 470, symbol R
- added R?: R, symbol R
- added U?: MX25L1606, symbol MX25L1606
- added W? (x3): TEST_1P, symbol TEST_1P
- added X1: USB_OTG, symbol USB_OTG
- added X?: CRYSTAL_SMD, symbol CRYSTAL_SMD
Connections:
- net labels added: +5V, D+, D-, LEFT, L_AC, PWRBUTTON, RIGHT, RX, RX_5V, R_AC, TX, VAA, VDD, VHIGH
- wire segments 8 -> 176

Commit message: Finished sch
Parts:
- added C?: 1uF, symbol C
- added GPIO?: GPIO_Breakout2, symbol GPIO_Breakout2
- added R? (x4): 100K, symbol R
- added x?: 19621, symbol 19621
Connections:
- net +5V: now also GPIO?.3 (VBUS)
- net GND: now also GPIO?.11 (GND), GPIO?.14 (GND), GPIO?.2 (GND), R?.1, x?.1 (Ring)
- net L_AC: now also x?.3 (Sleeve)
- net PWRBUTTON: now also C?.2, GPIO?.4 (PWRBUTTON), R?.2
- net RX_5V: now also GPIO?.6 (RX_5V)
- net R_AC: now also GPIO?.12 (R_AC), x?.4 (Ring)
- net TX: now also GPIO?.5 (TX)
- net VDD: now also R?.1, R?.1, R?.1
- net VHIGH: now also C?.1
- net GPIO13: now reaches IC?.17 (NFALE_/_GPIO0_13)
- net GPIO13: now also R?.2
- net GPIO_11: now reaches IC?.20 (NFWR_/_GPIO0_11)
- net GPIO_11: now also GPIO?.7 (GPIO_11), R?.2
- net CS: now reaches IC?.21 (CS2_/_GPIO0_14)
- net CS: now also IC?.22 (XCS_/_GPIO1_0), R?.2, U?.1 (CS), GPIO?.10 (CS), GPIO?.9 (GPIO_14), R?.2
- net at D?.2 (A): now also GPIO?.1 (VIN)
- new net GPIO_13: GPIO?.8 (GPIO_13)
- new net L_RC: GPIO?.13 (L_AC)
Other:
- moved on the sheet: W?
